Commit message: 实现了通过controller控制gazebo机械臂运动

File: my_arm_description/urdf/only_piper_description_gazebo.xacro (robot description, xacro)
@@ -23,19 +23,19 @@
       <geometry>
         <mesh
-          filename="package://my_arm_description/meshes/base_link.STL" />
-      </geometry>
-      <material
-        name="">
-        <color
-          rgba="0.792156862745098 0.819607843137255 0.933333333333333 1" />
-      </material>
-    </visual>
-    <collision>
-      <origin
-        xyz="0 0 0"
-        rpy="0 0 0" />
-      <geometry>
-        <mesh
-          filename="package://my_arm_description/meshes/base_link.STL" />
+          filename="file://$(find my_arm_description)/meshes/base_link.STL" />
+      </geometry>
+      <material
+        name="">
+        <color
+          rgba="0.792156862745098 0.819607843137255 0.933333333333333 1" />
+      </material>
+    </visual>
+    <collision>
+      <origin
+        xyz="0 0 0"
+        rpy="0 0 0" />
+      <geometry>
+        <mesh
+          filename="file://$(find my_arm_description)/meshes/base_link.STL" />
       </geometry>
     </collision>
@@ -54,19 +54,19 @@
       <geometry>
         <mesh
-          filename="package://my_arm_description/meshes/link1.STL" />
-      </geometry>
-      <material
-        name="">
-        <color
-          rgba="0.792156862745098 0.819607843137255 0.933333333333333 1" />
-      </material>
-    </visual>
-    <collision>
-      <origin
-        xyz="0 0 0"
-        rpy="0 0 0" />
-      <geometry>
-        <mesh
-          filename="package://my_arm_description/meshes/link1.STL" />
+          filename="file://$(find my_arm_description)/meshes/link1.STL" />
+      </geometry>
+      <material
+        name="">
+        <color
+          rgba="0.792156862745098 0.819607843137255 0.933333333333333 1" />
+      </material>
+    </visual>
+    <collision>
+      <origin
+        xyz="0 0 0"
+        rpy="0 0 0" />
+      <geometry>
+        <mesh
+          filename="file://$(find my_arm_description)/meshes/link1.STL" />
       </geometry>
     </collision>
@@ -103,19 +103,19 @@
       <geometry>
         <mesh
-          filename="package://my_arm_description/meshes/link2.STL" />
-      </geometry>
-      <material
-        name="">
-        <color
-          rgba="0.792156862745098 0.819607843137255 0.933333333333333 1" />
-      </material>
-    </visual>
-    <collision>
-      <origin
-        xyz="0 0 0"
-        rpy="0 0 0" />
-      <geometry>
-        <mesh
-          filename="package://my_arm_description/meshes/link2.STL" />
+          filename="file://$(find my_arm_description)/meshes/link2.STL" />
+      </geometry>
+      <material
+        name="">
+        <color
+          rgba="0.792156862745098 0.819607843137255 0.933333333333333 1" />
+      </material>
+    </visual>
+    <collision>
+      <origin
+        xyz="0 0 0"
+        rpy="0 0 0" />
+      <geometry>
+        <mesh
+          filename="file://$(find my_arm_description)/meshes/link2.STL" />
       </geometry>
     </collision>
@@ -153,19 +153,19 @@
       <geometry>
         <mesh
-          filename="package://my_arm_description/meshes/link3.STL" />
-      </geometry>
-      <material
-        name="">
-        <color
-          rgba="0.792156862745098 0.819607843137255 0.933333333333333 1" />
-      </material>
-    </visual>
-    <collision>
-      <origin
-        xyz="0 0 0"
-        rpy="0 0 0" />
-      <geometry>
-        <mesh
-          filename="package://my_arm_description/meshes/link3.STL" />
+          filename="file://$(find my_arm_description)/meshes/link3.STL" />
+      </geometry>
+      <material
+        name="">
+        <color
+          rgba="0.792156862745098 0.819607843137255 0.933333333333333 1" />
+      </material>
+    </visual>
+    <collision>
+      <origin
+        xyz="0 0 0"
+        rpy="0 0 0" />
+      <geometry>
+        <mesh
+          filename="file://$(find my_arm_description)/meshes/link3.STL" />
       </geometry>
     </collision>
@@ -203,19 +203,19 @@
       <geometry>
         <mesh
-          filename="package://my_arm_description/meshes/link4.STL" />
-      </geometry>
-      <material
-        name="">
-        <color
-          rgba="0.792156862745098 0.819607843137255 0.933333333333333 1" />
-      </material>
-    </visual>
-    <collision>
-      <origin
-        xyz="0 0 0"
-        rpy="0 0 0" />
-      <geometry>
-        <mesh
-          filename="package://my_arm_description/meshes/link4.STL" />
+          filename="file://$(find my_arm_description)/meshes/link4.STL" />
+      </geometry>
+      <material
+        name="">
+        <color
+          rgba="0.792156862745098 0.819607843137255 0.933333333333333 1" />
+      </material>
+    </visual>
+    <collision>
+      <origin
+        xyz="0 0 0"
+        rpy="0 0 0" />
+      <geometry>
+        <mesh
+          filename="file://$(find my_arm_description)/meshes/link4.STL" />
       </geometry>
     </collision>
@@ -252,19 +252,19 @@
       <geometry>
         <mesh
-          filename="package://my_arm_description/meshes/link5.STL" />
-      </geometry>
-      <material
-        name="">
-        <color
-          rgba="0.792156862745098 0.819607843137255 0.933333333333333 1" />
-      </material>
-    </visual>
-    <collision>
-      <origin
-        xyz="0 0 0"
-        rpy="0 0 0" />
-      <geometry>
-        <mesh
-          filename="package://my_arm_description/meshes/link5.STL" />
+          filename="file://$(find my_arm_description)/meshes/link5.STL" />
+      </geometry>
+      <material
+        name="">
+        <color
+          rgba="0.792156862745098 0.819607843137255 0.933333333333333 1" />
+      </material>
+    </visual>
+    <collision>
+      <origin
+        xyz="0 0 0"
+        rpy="0 0 0" />
+      <geometry>
+        <mesh
+          filename="file://$(find my_arm_description)/meshes/link5.STL" />
       </geometry>
     </collision>
@@ -301,5 +301,5 @@
       <geometry>
         <mesh
-          filename="package://my_arm_description/meshes/link6.STL" />
+          filename="file://$(find my_arm_description)/meshes/link6.STL" />
       </geometry>
       <material
@@ -315,5 +315,5 @@
       <geometry>
         <mesh
-          filename="package://my_arm_description/meshes/link6.STL" />
+          filename="file://$(find my_arm_description)/meshes/link6.STL" />
       </geometry>
     </collision>
@@ -336,56 +336,4 @@
       effort="100"
       velocity="3" />
-  </joint>
-  <!--gripper link-->
-  <link
-    name="gripper_base">
-    <inertial>
-      <origin
-        xyz="-0.000183807162235591 8.05033155577911E-05 0.0321436689908876"
-        rpy="0 0 0" />
-      <mass
-        value="0.1" />
-      <inertia
-        ixx="0.00092934"
-        ixy="0.00000034"
-        ixz="-0.00000738"
-        iyy="0.00071447"
-        iyz="0.00000005"
-        izz="0.00039442" />
-    </inertial>
-    <visual>
-      <origin
-        xyz="0 0 0"
-        rpy="0 0 0" />
-      <geometry>
-        <mesh
-          filename="package://my_arm_description/meshes/my_gripper.STL" />
-      </geometry>
-      <material
-        name="">
-        <color
-          rgba="0.792156862745098 0.819607843137255 0.933333333333333 1" />
-      </material>
-    </visual>
-    <collision>
-      <origin
-        xyz="0 0 0"
-        rpy="0 0 0" />
-      <geometry>
-        <mesh
-          filename="package://my_arm_description/meshes/my_gripper.STL" />
-      </geometry>
-    </collision>
-  </link>
-  <joint
-    name="joint6_to_gripper_base"
-    type="fixed">
-    <origin
-      xyz="0 0 0"
-      rpy="0 0 0" />
-    <parent
-      link="link6" />
-    <child
-      link="gripper_base" />
   </joint>
   <!-- <gazebo reference="base_link">
@@ -427,5 +375,4 @@
           </state_interface>
           <state_interface name="velocity"/>
-          <state_interface name="effort"/>
       </joint>
       <joint name="joint2">
@@ -438,5 +385,4 @@
           </state_interface>
           <state_interface name="velocity"/>
-          <state_interface name="effort"/>
       </joint>
       <joint name="joint3">
@@ -449,5 +395,4 @@
           </state_interface>
           <state_interface name="velocity"/>
-          <state_interface name="effort"/>
       </joint>
       <joint name="joint4">
@@ -460,5 +405,4 @@
           </state_interface>
           <state_interface name="velocity"/>
-          <state_interface name="effort"/>
       </joint>
       <joint name="joint5">
@@ -471,5 +415,4 @@
           </state_interface>
           <state_interface name="velocity"/>
-          <state_interface name="effort"/>
       </joint>
       <joint name="joint6">
@@ -482,5 +425,4 @@
           </state_interface>
           <state_interface name="velocity"/>
-          <state_interface name="effort"/>
       </joint>
   </ros2_control>

File: my_arm_description/urdf/piper_with_my_gripper_description_gazebo.urdf.xacro (robot description, xacro)
@@ -23,19 +23,19 @@
       <geometry>
         <mesh
-          filename="package://my_arm_description/meshes/base_link.STL" />
-      </geometry>
-      <material
-        name="">
-        <color
-          rgba="0.792156862745098 0.819607843137255 0.933333333333333 1" />
-      </material>
-    </visual>
-    <collision>
-      <origin
-        xyz="0 0 0"
-        rpy="0 0 0" />
-      <geometry>
-        <mesh
-          filename="package://my_arm_description/meshes/base_link.STL" />
+          filename="file://$(find my_arm_description)/meshes/base_link.STL" />
+      </geometry>
+      <material
+        name="">
+        <color
+          rgba="0.792156862745098 0.819607843137255 0.933333333333333 1" />
+      </material>
+    </visual>
+    <collision>
+      <origin
+        xyz="0 0 0"
+        rpy="0 0 0" />
+      <geometry>
+        <mesh
+          filename="file://$(find my_arm_description)/meshes/base_link.STL" />
       </geometry>
     </collision>
@@ -54,19 +54,19 @@
       <geometry>
         <mesh
-          filename="package://my_arm_description/meshes/link1.STL" />
-      </geometry>
-      <material
-        name="">
-        <color
-          rgba="0.792156862745098 0.819607843137255 0.933333333333333 1" />
-      </material>
-    </visual>
-    <collision>
-      <origin
-        xyz="0 0 0"
-        rpy="0 0 0" />
-      <geometry>
-        <mesh
-          filename="package://my_arm_description/meshes/link1.STL" />
+          filename="file://$(find my_arm_description)/meshes/link1.STL" />
+      </geometry>
+      <material
+        name="">
+        <color
+          rgba="0.792156862745098 0.819607843137255 0.933333333333333 1" />
+      </material>
+    </visual>
+    <collision>
+      <origin
+        xyz="0 0 0"
+        rpy="0 0 0" />
+      <geometry>
+        <mesh
+          filename="file://$(find my_arm_description)/meshes/link1.STL" />
       </geometry>
     </collision>
@@ -103,19 +103,19 @@
       <geometry>
         <mesh
-          filename="package://my_arm_description/meshes/link2.STL" />
-      </geometry>
-      <material
-        name="">
-        <color
-          rgba="0.792156862745098 0.819607843137255 0.933333333333333 1" />
-      </material>
-    </visual>
-    <collision>
-      <origin
-        xyz="0 0 0"
-        rpy="0 0 0" />
-      <geometry>
-        <mesh
-          filename="package://my_arm_description/meshes/link2.STL" />
+          filename="file://$(find my_arm_description)/meshes/link2.STL" />
+      </geometry>
+      <material
+        name="">
+        <color
+          rgba="0.792156862745098 0.819607843137255 0.933333333333333 1" />
+      </material>
+    </visual>
+    <collision>
+      <origin
+        xyz="0 0 0"
+        rpy="0 0 0" />
+      <geometry>
+        <mesh
+          filename="file://$(find my_arm_description)/meshes/link2.STL" />
       </geometry>
     </collision>
@@ -153,19 +153,19 @@
       <geometry>
         <mesh
-          filename="package://my_arm_description/meshes/link3.STL" />
-      </geometry>
-      <material
-        name="">
-        <color
-          rgba="0.792156862745098 0.819607843137255 0.933333333333333 1" />
-      </material>
-    </visual>
-    <collision>
-      <origin
-        xyz="0 0 0"
-        rpy="0 0 0" />
-      <geometry>
-        <mesh
-          filename="package://my_arm_description/meshes/link3.STL" />
+          filename="file://$(find my_arm_description)/meshes/link3.STL" />
+      </geometry>
+      <material
+        name="">
+        <color
+          rgba="0.792156862745098 0.819607843137255 0.933333333333333 1" />
+      </material>
+    </visual>
+    <collision>
+      <origin
+        xyz="0 0 0"
+        rpy="0 0 0" />
+      <geometry>
+        <mesh
+          filename="file://$(find my_arm_description)/meshes/link3.STL" />
       </geometry>
     </collision>
@@ -203,19 +203,19 @@
       <geometry>
         <mesh
-          filename="package://my_arm_description/meshes/link4.STL" />
-      </geometry>
-      <material
-        name="">
-        <color
-          rgba="0.792156862745098 0.819607843137255 0.933333333333333 1" />
-      </material>
-    </visual>
-    <collision>
-      <origin
-        xyz="0 0 0"
-        rpy="0 0 0" />
-      <geometry>
-        <mesh
-          filename="package://my_arm_description/meshes/link4.STL" />
+          filename="file://$(find my_arm_description)/meshes/link4.STL" />
+      </geometry>
+      <material
+        name="">
+        <color
+          rgba="0.792156862745098 0.819607843137255 0.933333333333333 1" />
+      </material>
+    </visual>
+    <collision>
+      <origin
+        xyz="0 0 0"
+        rpy="0 0 0" />
+      <geometry>
+        <mesh
+          filename="file://$(find my_arm_description)/meshes/link4.STL" />
       </geometry>
     </collision>
@@ -252,19 +252,19 @@
       <geometry>
         <mesh
-          filename="package://my_arm_description/meshes/link5.STL" />
-      </geometry>
-      <material
-        name="">
-        <color
-          rgba="0.792156862745098 0.819607843137255 0.933333333333333 1" />
-      </material>
-    </visual>
-    <collision>
-      <origin
-        xyz="0 0 0"
-        rpy="0 0 0" />
-      <geometry>
-        <mesh
-          filename="package://my_arm_description/meshes/link5.STL" />
+          filename="file://$(find my_arm_description)/meshes/link5.STL" />
+      </geometry>
+      <material
+        name="">
+        <color
+          rgba="0.792156862745098 0.819607843137255 0.933333333333333 1" />
+      </material>
+    </visual>
+    <collision>
+      <origin
+        xyz="0 0 0"
+        rpy="0 0 0" />
+      <geometry>
+        <mesh
+          filename="file://$(find my_arm_description)/meshes/link5.STL" />
       </geometry>
     </collision>
@@ -301,5 +301,5 @@
       <geometry>
         <mesh
-          filename="package://my_arm_description/meshes/link6.STL" />
+          filename="file://$(find my_arm_description)/meshes/link6.STL" />
       </geometry>
       <material
@@ -315,5 +315,5 @@
       <geometry>
         <mesh
-          filename="package://my_arm_description/meshes/link6.STL" />
+          filename="file://$(find my_arm_description)/meshes/link6.STL" />
       </geometry>
     </collision>
@@ -355,5 +355,5 @@
         rpy="0 0 0" />
       <geometry>
-        <mesh filename="package://my_arm_description/meshes/my_gripper.STL" />
+        <mesh filename="file://$(find my_arm_description)/meshes/my_gripper.STL" />
       </geometry>
       <material
@@ -368,5 +368,5 @@
       <geometry>
         <mesh
-          filename="package://my_arm_description/meshes/my_gripper.STL" />
+          filename="file://$(find my_arm_description)/meshes/my_gripper.STL" />
       </geometry>
     </collision>
